Commit message: change robot model

File: my_robot/urdf/my_robot.xacro (robot description, xacro)
@@ -1,48 +1,54 @@
-<?xml version='1.0'?>
+<?xml version="1.0"?>
 <robot name="my_robot" xmlns:xacro="http://www.ros.org/wiki/xacro">
   <xacro:include filename="$(find my_robot)/urdf/my_robot.gazebo" />
+  <material name="blue">
+    <color rgba="0 0 0.8 1"/>
+  </material>
+  <material name="black">
+    <color rgba="0 0 0 1"/>
+  </material>
+  <material name="white">
+    <color rgba="1 1 1 1"/>
+  </material>
   <link name="robot_footprint"></link>
   <joint name="robot_footprint_joint" type="fixed">
     <origin xyz="0 0 0" rpy="0 0 0" />
     <parent link="robot_footprint"/>
-    <child link="chassis" />
+    <child link="base_link" />
   </joint>
-  <link name='chassis'>
-    <pose>0 0 0.1 0 0 0</pose>
-    <inertial>
-      <mass value="15.0"/>
-      <origin xyz="0.0 0 0" rpy=" 0 0 0"/>
-      <inertia
-          ixx="0.1" ixy="0" ixz="0"
-          iyy="0.1" iyz="0"
-          izz="0.1"
-      />
-    </inertial>
-    <collision name='collision'>
-      <origin xyz="0 0 0" rpy=" 0 0 0"/>
+  <link name="base_link">
+    <pose>0 0 0.05 0 0 0</pose>
+    <visual>
       <geometry>
-        <box size=".4 .2 .1"/>
+        <cylinder length="0.6" radius="0.2"/>
+      </geometry>
+      <material name="blue"/>
+    </visual>
+    <collision>
+      <geometry>
+        <cylinder length="0.6" radius="0.2"/>
       </geometry>
     </collision>
-    <visual name='chassis_visual'>
-      <origin xyz="0 0 0" rpy=" 0 0 0"/>
+  </link>
+  <link name="box">
+    <visual>
       <geometry>
-        <box size=".4 .2 .1"/>
+        <box size="0.2 0.4 0.6"/>
       </geometry>
+      <material name="blue"/>
     </visual>
-    <collision name='back_caster_collision'>
-      <origin xyz="-0.15 0 -0.05" rpy=" 0 0 0"/>
+    <collision>
       <geometry>
-        <sphere radius="0.0499"/>
+        <box size="0.2 0.4 0.6"/>
       </geometry>
     </collision>
-    <visual name='back_caster_visual'>
-      <origin xyz="-0.15 0 -0.05" rpy=" 0 0 0"/>
-      <geometry>
-        <sphere radius="0.05"/>
-      </geometry>
-    </visual>
+  </link>
+  <joint name="body_joint" type="fixed">
+    <parent link="base_link"/>
+    <child link="box"/>
+    <origin xyz="-0.1 0 0"/>
+  </joint>
+  <link name="front_caster">
     <collision name='front_caster_collision'>
-      <origin xyz="0.15 0 -0.05" rpy=" 0 0 0"/>
       <geometry>
         <sphere radius="0.0499"/>
@@ -50,5 +56,4 @@
     </collision>
     <visual name='front_caster_visual'>
-      <origin xyz="0.15 0 -0.05" rpy=" 0 0 0"/>
       <geometry>
         <sphere radius="0.05"/>
@@ -56,73 +61,93 @@
     </visual>
   </link>
-  <link name='left_wheel'>
-    <inertial>
-      <mass value="5.0"/>
-      <origin xyz="0.0 0 0" rpy=" 0 0 0"/>
-      <inertia
-          ixx="0.1" ixy="0" ixz="0"
-          iyy="0.1" iyz="0"
-          izz="0.1"
-      />
-    </inertial>
-    <collision name='collision'>
-      <origin xyz="0 0 0" rpy=" 0 1.5707 1.5707"/>
+  <joint name="front_caster_joint" type="fixed">
+    <parent link="base_link"/>
+    <child link="front_caster"/>
+    <origin xyz="0.1 0 0.3"/>
+  </joint>
+   <link name="head">
+    <visual>
       <geometry>
-        <cylinder radius=".1" length=".05"/>
+        <sphere radius="0.2"/>
+      </geometry>
+      <material name="white"/>
+    </visual>
+    <collision>
+      <geometry>
+        <sphere radius="0.2"/>
       </geometry>
     </collision>
-    <visual name='chassis_visual'>
-      <origin xyz="0 0 0" rpy=" 0 1.5707 1.5707"/>
+  </link>
+  <joint name="head_swivel" type="fixed">
+    <parent link="base_link"/>
+    <child link="head"/>
+    <origin xyz="0 0 0.3"/>
+  </joint>
+  <link name="camera">
+    <visual>
       <geometry>
-        <cylinder radius=".1" length=".05"/>
+        <box size="0.08 0.08 0.08"/>
       </geometry>
+      <material name="blue"/>
     </visual>
-  </link>
-  <link name='right_wheel'>
-    <inertial>
-      <mass value="5.0"/>
-      <origin xyz="0.0 0 0" rpy=" 0 0 0"/>
-      <inertia
-          ixx="0.1" ixy="0" ixz="0"
-          iyy="0.1" iyz="0"
-          izz="0.1"
-      />
-    </inertial>
-    <collision name='collision'>
-      <origin xyz="0 0 0" rpy=" 0 1.5707 1.5707"/>
+    <collision>
       <geometry>
-        <cylinder radius=".1" length=".05"/>
+        <box size="0.08 0.08 0.08"/>
       </geometry>
     </collision>
-    <visual name='chassis_visual'>
-      <origin xyz="0 0 0" rpy=" 0 1.5707 1.5707"/>
+  </link>
+  <joint name="camera_joint" type="fixed">
+    <parent link="head"/>
+    <child link="camera"/>
+    <origin xyz="0.1814 0 0.1414"/>
+  </joint>
+  <link name="right_wheel">
+    <visual>
+      <origin rpy="1.57075 0 0" xyz="0 0 0"/>
       <geometry>
-        <cylinder radius=".1" length=".05"/>
+        <cylinder length="0.05" radius="0.1"/>
       </geometry>
+      <material name="black"/>
     </visual>
-  </link>
-  <link name='camera'>
-    <inertial>
-      <mass value="0.1"/>
-      <origin xyz="0.05 0.05 0.05" rpy=" 0 0 0"/>
-      <inertia
-          ixx="1e-6" ixy="0" ixz="0"
-          iyy="1e-6" iyz="0"
-          izz="1e-6"
-      />
-    </inertial>
-    <collision name='camera_collision'>
-      <origin xyz="0 0 0" rpy="0 0 0"/>
+    <collision>
+      <origin rpy="1.57075 0 0" xyz="0 0 0"/>
       <geometry>
-        <box size="0.05 0.05 0.05"/>
+        <cylinder length="0.05" radius="0.1"/>
       </geometry>
     </collision>
-    <visual name='camera_visual'>
-      <origin xyz="0 0 0" rpy="0 0 0"/>
+  </link>
+  <joint name="right_wheel_joint" type="continuous">
+    <parent link="box"/>
+    <child link="right_wheel"/>
+    <origin xyz="0 0.2 -0.25"/>
+    <axis xyz="0 1 0" rpy="0 0 0"/>
+    <limit effort="10000" velocity="1000"/>
+    <dynamics damping="1.0" friction="1.0"/>
+  </joint>
+  <link name="left_wheel">
+    <visual>
+      <origin rpy="1.57075 0 0" xyz="0 0 0"/>
       <geometry>
-        <box size="0.05 0.05 0.05"/>
+        <cylinder length="0.05" radius="0.1"/>
       </geometry>
+      <material name="black"/>
+      <origin rpy="0 0 0" xyz="0 0 0"/>
     </visual>
+    <collision>
+      <origin rpy="1.57075 0 0" xyz="0 0 0"/>
+      <geometry>
+        <cylinder length="0.05" radius="0.1"/>
+      </geometry>
+      <origin rpy="0 0 0" xyz="0 0 0"/>
+    </collision>
   </link>
+  <joint name="left_wheel_joint" type="continuous">
+    <parent link="box"/>
+    <child link="left_wheel"/>
+    <origin xyz="0 -0.2 -0.25"/>
+    <axis xyz="0 1 0" rpy="0 0 0"/>
+    <limit effort="10000" velocity="1000"/>
+    <dynamics damping="1.0" friction="1.0"/>
+  </joint>
   <link name='hokuyo'>
     <inertial>
@@ -148,30 +173,8 @@
     </visual>
   </link>
-  <joint type="continuous" name="left_wheel_hinge">
-    <origin xyz="0 0.15 0" rpy="0 0 0"/>
-    <child link="left_wheel"/>
-    <parent link="chassis"/>
-    <axis xyz="0 1 0" rpy="0 0 0"/>
-    <limit effort="10000" velocity="1000"/>
-    <dynamics damping="1.0" friction="1.0"/>
-  </joint>
-  <joint type="continuous" name="right_wheel_hinge">
-    <origin xyz="0 -0.15 0" rpy="0 0 0"/>
-    <child link="right_wheel"/>
-    <parent link="chassis"/>
-    <axis xyz="0 1 0" rpy="0 0 0"/>
-    <limit effort="10000" velocity="1000"/>
-    <dynamics damping="1.0" friction="1.0"/>
-  </joint>
-  <joint type="fixed" name="camera_joint">
-    <origin xyz="0.2 0 0" rpy="0 0 0"/>
-    <child link="camera"/>
-    <parent link="chassis"/>
-    <axis xyz="0 1 0" rpy="0 0 0"/>
-  </joint>
-   <joint type="fixed" name="hokuyo_joint">
-    <origin xyz="0.15 0 0.1" rpy="0 0 0"/>
+  <joint type="fixed" name="hokuyo_joint">
+    <origin xyz="0.0 0 0.2" rpy="0 0 0"/>
     <child link="hokuyo"/>
-    <parent link="chassis"/>
+    <parent link="head"/>
     <axis xyz="0 1 0" rpy="0 0 0"/>
   </joint>

Commit message: modify my_robot.xacro

File: my_robot/urdf/my_robot.xacro (robot description, xacro)
@@ -19,4 +19,13 @@
   <link name="base_link">
     <pose>0 0 0.05 0 0 0</pose>
+    <inertial>
+      <mass value="15.0"/>
+      <origin xyz="0.0 0 0" rpy=" 0 0 0"/>
+      <inertia
+          ixx="0.1" ixy="0" ixz="0"
+          iyy="0.1" iyz="0"
+          izz="0.1"
+      />
+    </inertial>
     <visual>
       <geometry>
@@ -44,5 +53,5 @@
     </collision>
   </link>
-  <joint name="body_joint" type="fixed">
+  <joint name="box_joint" type="fixed">
     <parent link="base_link"/>
     <child link="box"/>
@@ -103,15 +112,24 @@
   </joint>
   <link name="right_wheel">
-    <visual>
-      <origin rpy="1.57075 0 0" xyz="0 0 0"/>
-      <geometry>
-        <cylinder length="0.05" radius="0.1"/>
+    <inertial>
+      <mass value="5.0"/>
+      <origin xyz="0.0 0 0" rpy=" 0 0 0"/>
+      <inertia
+          ixx="0.1" ixy="0" ixz="0"
+          iyy="0.1" iyz="0"
+          izz="0.1"
+      />
+    </inertial>
+    <visual>
+      <origin rpy="0 1.57075 1.57075" xyz="0 0 0"/>
+      <geometry>
+        <cylinder length="0.1" radius="0.1"/>
       </geometry>
       <material name="black"/>
     </visual>
     <collision>
-      <origin rpy="1.57075 0 0" xyz="0 0 0"/>
-      <geometry>
-        <cylinder length="0.05" radius="0.1"/>
+      <origin rpy="0 1.57075 1.57075" xyz="0 0 0"/>
+      <geometry>
+        <cylinder length="0.1" radius="0.1"/>
       </geometry>
     </collision>
@@ -126,8 +144,17 @@
   </joint>
   <link name="left_wheel">
-    <visual>
-      <origin rpy="1.57075 0 0" xyz="0 0 0"/>
-      <geometry>
-        <cylinder length="0.05" radius="0.1"/>
+    <inertial>
+      <mass value="5.0"/>
+      <origin xyz="0.0 0 0" rpy=" 0 0 0"/>
+      <inertia
+          ixx="0.1" ixy="0" ixz="0"
+          iyy="0.1" iyz="0"
+          izz="0.1"
+      />
+    </inertial>
+    <visual>
+      <origin rpy="0 1.57075 1.57075" xyz="0 0 0"/>
+      <geometry>
+        <cylinder length="0.1" radius="0.1"/>
       </geometry>
       <material name="black"/>
@@ -135,7 +162,7 @@
     </visual>
     <collision>
-      <origin rpy="1.57075 0 0" xyz="0 0 0"/>
-      <geometry>
-        <cylinder length="0.05" radius="0.1"/>
+      <origin rpy="0 1.57075 1.57075" xyz="0 0 0"/>
+      <geometry>
+        <cylinder length="0.1" radius="0.1"/>
       </geometry>
       <origin rpy="0 0 0" xyz="0 0 0"/>

Commit message: new robot model

File: my_robot/urdf/my_robot.xacro (robot description, xacro)
@@ -28,5 +28,6 @@
       />
     </inertial>
-    <visual>
+    <visual name="body_visual">
+      <origin xyz="0 0 0" rpy=" 0 0 0"/>
       <geometry>
         <cylinder length="0.6" radius="0.2"/>
@@ -34,30 +35,12 @@
       <material name="blue"/>
     </visual>
-    <collision>
+    <collision name="body_collision">
+      <origin xyz="0 0 0" rpy=" 0 0 0"/>
       <geometry>
         <cylinder length="0.6" radius="0.2"/>
       </geometry>
     </collision>
-  </link>
-  <link name="box">
-    <visual>
-      <geometry>
-        <box size="0.2 0.4 0.6"/>
-      </geometry>
-      <material name="blue"/>
-    </visual>
-    <collision>
-      <geometry>
-        <box size="0.2 0.4 0.6"/>
-      </geometry>
-    </collision>
-  </link>
-  <joint name="box_joint" type="fixed">
-    <parent link="base_link"/>
-    <child link="box"/>
-    <origin xyz="-0.1 0 0"/>
-  </joint>
-  <link name="front_caster">
     <collision name='front_caster_collision'>
+      <origin xyz="-0.15 0 -0.3" rpy=" 0 0 0"/>
       <geometry>
         <sphere radius="0.0499"/>
@@ -65,4 +48,17 @@
     </collision>
     <visual name='front_caster_visual'>
+      <origin xyz="-0.15 0 -0.3" rpy=" 0 0 0"/>
+      <geometry>
+        <sphere radius="0.05"/>
+      </geometry>
+    </visual>
+    <collision name='back_caster_collision'>
+      <origin xyz="0.15 0 -0.3" rpy=" 0 0 0"/>
+      <geometry>
+        <sphere radius="0.0499"/>
+      </geometry>
+    </collision>
+    <visual name='back_caster_visual'>
+      <origin xyz="0.15 0 -0.3" rpy=" 0 0 0"/>
       <geometry>
         <sphere radius="0.05"/>
@@ -70,9 +66,4 @@
     </visual>
   </link>
-  <joint name="front_caster_joint" type="fixed">
-    <parent link="base_link"/>
-    <child link="front_caster"/>
-    <origin xyz="0.1 0 0.3"/>
-  </joint>
    <link name="head">
     <visual>
@@ -136,5 +127,5 @@
   </link>
   <joint name="right_wheel_joint" type="continuous">
-    <parent link="box"/>
+    <parent link="base_link"/>
     <child link="right_wheel"/>
     <origin xyz="0 0.2 -0.25"/>
@@ -170,5 +161,5 @@
   </link>
   <joint name="left_wheel_joint" type="continuous">
-    <parent link="box"/>
+    <parent link="base_link"/>
     <child link="left_wheel"/>
     <origin xyz="0 -0.2 -0.25"/>
